Commit message: anisotropic with slower wriggling speed

File: examples/snake/bb_snake.urdf (robot description, URDF)
Before this commit: robot bb_snake, 83 links, 82 joints
Links:
- link act0Seg0: mass 0.3 -> 0.595; geometry collision box size=0.11 0.12 0.0245; visual box size=0.11 0.12 0.0245
- link act0Seg1: mass 0.3 -> 0.595; geometry collision box size=0.11 0.12 0.049; visual box size=0.11 0.12 0.049
- link act0Seg10: mass 0.3 -> 0.595; geometry collision box size=0.11 0.12 0.049; visual box size=0.11 0.12 0.049
- link act0Seg10helper_shape: mass 0.0003 -> 0.0005949999999999999; geometry collision cylinder length=0.12 radius=0.055; visual cylinder length=0.12 radius=0.055
- link act0Seg11: mass 0.3 -> 0.595; geometry collision box size=0.11 0.12 0.049; visual box size=0.11 0.12 0.049
- link act0Seg11helper_shape: mass 0.0003 -> 0.0005949999999999999; geometry collision cylinder length=0.11 radius=0.06; visual cylinder length=0.11 radius=0.06
- link act0Seg12: mass 0.3 -> 0.595; geometry collision box size=0.11 0.12 0.049; visual box size=0.11 0.12 0.049
- link act0Seg12helper_shape: mass 0.0003 -> 0.0005949999999999999; geometry collision cylinder length=0.12 radius=0.055; visual cylinder length=0.12 radius=0.055
- link act0Seg13: mass 0.3 -> 0.595; geometry collision box size=0.11 0.12 0.049; visual box size=0.11 0.12 0.049
- link act0Seg13helper_shape: mass 0.0003 -> 0.0005949999999999999; geometry collision cylinder length=0.11 radius=0.06; visual cylinder length=0.11 radius=0.06
- link act0Seg14: mass 0.3 -> 0.595; geometry collision box size=0.11 0.12 0.049; visual box size=0.11 0.12 0.049
- link act0Seg14helper_shape: mass 0.0003 -> 0.0005949999999999999; geometry collision cylinder length=0.12 radius=0.055; visual cylinder length=0.12 radius=0.055
- link act0Seg15: mass 0.3 -> 0.595; geometry collision box size=0.11 0.12 0.049; visual box size=0.11 0.12 0.049
- link act0Seg15helper_shape: mass 0.0003 -> 0.0005949999999999999; geometry collision cylinder length=0.11 radius=0.06; visual cylinder length=0.11 radius=0.06
- link act0Seg16: mass 0.3 -> 0.595; geometry collision box size=0.11 0.12 0.049; visual box size=0.11 0.12 0.049
- link act0Seg16helper_shape: mass 0.0003 -> 0.0005949999999999999; geometry collision cylinder length=0.12 radius=0.055; visual cylinder length=0.12 radius=0.055
- link act0Seg17: mass 0.3 -> 0.595; geometry collision box size=0.11 0.12 0.049; visual box size=0.11 0.12 0.049
- link act0Seg17helper_shape: mass 0.0003 -> 0.0005949999999999999; geometry collision cylinder length=0.11 radius=0.06; visual cylinder length=0.11 radius=0.06
- link act0Seg18: mass 0.3 -> 0.595; geometry collision box size=0.11 0.12 0.049; visual box size=0.11 0.12 0.049
- link act0Seg18helper_shape: mass 0.0003 -> 0.0005949999999999999; geometry collision cylinder length=0.12 radius=0.055; visual cylinder length=0.12 radius=0.055
- link act0Seg19: mass 0.3 -> 0.595; geometry collision box size=0.11 0.12 0.049; visual box size=0.11 0.12 0.049
- link act0Seg19helper_shape: mass 0.0003 -> 0.0005949999999999999; geometry collision cylinder length=0.11 radius=0.06; visual cylinder length=0.11 radius=0.06
- link act0Seg1helper_shape: mass 0.0003 -> 0.0005949999999999999; geometry collision cylinder length=0.11 radius=0.06; visual cylinder length=0.11 radius=0.06
- link act0Seg2: mass 0.3 -> 0.595; geometry collision box size=0.11 0.12 0.049; visual box size=0.11 0.12 0.049
- link act0Seg20: mass 0.3 -> 0.595; geometry collision box size=0.11 0.12 0.0245; visual box size=0.11 0.12 0.0245
- link act0Seg20helper_shape: mass 0.0003 -> 0.0005949999999999999; geometry collision cylinder length=0.12 radius=0.055; visual cylinder length=0.12 radius=0.055
- link act0Seg2helper_shape: mass 0.0003 -> 0.0005949999999999999; geometry collision cylinder length=0.12 radius=0.055; visual cylinder length=0.12 radius=0.055
- link act0Seg3: mass 0.3 -> 0.595; geometry collision box size=0.11 0.12 0.049; visual box size=0.11 0.12 0.049
- link act0Seg3helper_shape: mass 0.0003 -> 0.0005949999999999999; geometry collision cylinder length=0.11 radius=0.06; visual cylinder length=0.11 radius=0.06
- link act0Seg4: mass 0.3 -> 0.595; geometry collision box size=0.11 0.12 0.049; visual box size=0.11 0.12 0.049
- link act0Seg4helper_shape: mass 0.0003 -> 0.0005949999999999999; geometry collision cylinder length=0.12 radius=0.055; visual cylinder length=0.12 radius=0.055
- link act0Seg5: mass 0.3 -> 0.595; geometry collision box size=0.11 0.12 0.049; visual box size=0.11 0.12 0.049
- link act0Seg5helper_shape: mass 0.0003 -> 0.0005949999999999999; geometry collision cylinder length=0.11 radius=0.06; visual cylinder length=0.11 radius=0.06
- link act0Seg6: mass 0.3 -> 0.595; geometry collision box size=0.11 0.12 0.049; visual box size=0.11 0.12 0.049
- link act0Seg6helper_shape: mass 0.0003 -> 0.0005949999999999999; geometry collision cylinder length=0.12 radius=0.055; visual cylinder length=0.12 radius=0.055
- link act0Seg7: mass 0.3 -> 0.595; geometry collision box size=0.11 0.12 0.049; visual box size=0.11 0.12 0.049
- link act0Seg7helper_shape: mass 0.0003 -> 0.0005949999999999999; geometry collision cylinder length=0.11 radius=0.06; visual cylinder length=0.11 radius=0.06
- link act0Seg8: mass 0.3 -> 0.595; geometry collision box size=0.11 0.12 0.049; visual box size=0.11 0.12 0.049
- link act0Seg8helper_shape: mass 0.0003 -> 0.0005949999999999999; geometry collision cylinder length=0.12 radius=0.055; visual cylinder length=0.12 radius=0.055
- link act0Seg9: mass 0.3 -> 0.595; geometry collision box size=0.11 0.12 0.049; visual box size=0.11 0.12 0.049
- link act0Seg9helper_shape: mass 0.0003 -> 0.0005949999999999999; geometry collision cylinder length=0.11 radius=0.06; visual cylinder length=0.11 radius=0.06
- link act1Seg0: mass 0.3 -> 0.595; geometry collision box size=0.11 0.12 0.0245; visual box size=0.11 0.12 0.0245
- link act1Seg1: mass 0.3 -> 0.595; geometry collision box size=0.11 0.12 0.049; visual box size=0.11 0.12 0.049
- link act1Seg10: mass 0.3 -> 0.595; geometry collision box size=0.11 0.12 0.049; visual box size=0.11 0.12 0.049
- link act1Seg10helper_shape: mass 0.0003 -> 0.0005949999999999999; geometry collision cylinder length=0.12 radius=0.055; visual cylinder length=0.12 radius=0.055
- link act1Seg11: mass 0.3 -> 0.595; geometry collision box size=0.11 0.12 0.049; visual box size=0.11 0.12 0.049
- link act1Seg11helper_shape: mass 0.0003 -> 0.0005949999999999999; geometry collision cylinder length=0.11 radius=0.06; visual cylinder length=0.11 radius=0.06
- link act1Seg12: mass 0.3 -> 0.595; geometry collision box size=0.11 0.12 0.049; visual box size=0.11 0.12 0.049
- link act1Seg12helper_shape: mass 0.0003 -> 0.0005949999999999999; geometry collision cylinder length=0.12 radius=0.055; visual cylinder length=0.12 radius=0.055
- link act1Seg13: mass 0.3 -> 0.595; geometry collision box size=0.11 0.12 0.049; visual box size=0.11 0.12 0.049
- link act1Seg13helper_shape: mass 0.0003 -> 0.0005949999999999999; geometry collision cylinder length=0.11 radius=0.06; visual cylinder length=0.11 radius=0.06
- link act1Seg14: mass 0.3 -> 0.595; geometry collision box size=0.11 0.12 0.049; visual box size=0.11 0.12 0.049
- link act1Seg14helper_shape: mass 0.0003 -> 0.0005949999999999999; geometry collision cylinder length=0.12 radius=0.055; visual cylinder length=0.12 radius=0.055
- link act1Seg15: mass 0.3 -> 0.595; geometry collision box size=0.11 0.12 0.049; visual box size=0.11 0.12 0.049
- link act1Seg15helper_shape: mass 0.0003 -> 0.0005949999999999999; geometry collision cylinder length=0.11 radius=0.06; visual cylinder length=0.11 radius=0.06
- link act1Seg16: mass 0.3 -> 0.595; geometry collision box size=0.11 0.12 0.049; visual box size=0.11 0.12 0.049
- link act1Seg16helper_shape: mass 0.0003 -> 0.0005949999999999999; geometry collision cylinder length=0.12 radius=0.055; visual cylinder length=0.12 radius=0.055
- link act1Seg17: mass 0.3 -> 0.595; geometry collision box size=0.11 0.12 0.049; visual box size=0.11 0.12 0.049
- link act1Seg17helper_shape: mass 0.0003 -> 0.0005949999999999999; geometry collision cylinder length=0.11 radius=0.06; visual cylinder length=0.11 radius=0.06
- link act1Seg18: mass 0.3 -> 0.595; geometry collision box size=0.11 0.12 0.049; visual box size=0.11 0.12 0.049
- link act1Seg18helper_shape: mass 0.0003 -> 0.0005949999999999999; geometry collision cylinder length=0.12 radius=0.055; visual cylinder length=0.12 radius=0.055
- link act1Seg19: mass 0.3 -> 0.595; geometry collision box size=0.11 0.12 0.049; visual box size=0.11 0.12 0.049
- link act1Seg19helper_shape: mass 0.0003 -> 0.0005949999999999999; geometry collision cylinder length=0.11 radius=0.06; visual cylinder length=0.11 radius=0.06
- link act1Seg1helper_shape: mass 0.0003 -> 0.0005949999999999999; geometry collision cylinder length=0.11 radius=0.06; visual cylinder length=0.11 radius=0.06
- link act1Seg2: mass 0.3 -> 0.595; geometry collision box size=0.11 0.12 0.049; visual box size=0.11 0.12 0.049
- link act1Seg20: mass 0.3 -> 0.595; geometry collision box size=0.11 0.12 0.0245; visual box size=0.11 0.12 0.0245
- link act1Seg20helper_shape: mass 0.0003 -> 0.0005949999999999999; geometry collision cylinder length=0.12 radius=0.055; visual cylinder length=0.12 radius=0.055
- link act1Seg2helper_shape: mass 0.0003 -> 0.0005949999999999999; geometry collision cylinder length=0.12 radius=0.055; visual cylinder length=0.12 radius=0.055
- link act1Seg3: mass 0.3 -> 0.595; geometry collision box size=0.11 0.12 0.049; visual box size=0.11 0.12 0.049
- link act1Seg3helper_shape: mass 0.0003 -> 0.0005949999999999999; geometry collision cylinder length=0.11 radius=0.06; visual cylinder length=0.11 radius=0.06
- link act1Seg4: mass 0.3 -> 0.595; geometry collision box size=0.11 0.12 0.049; visual box size=0.11 0.12 0.049
- link act1Seg4helper_shape: mass 0.0003 -> 0.0005949999999999999; geometry collision cylinder length=0.12 radius=0.055; visual cylinder length=0.12 radius=0.055
- link act1Seg5: mass 0.3 -> 0.595; geometry collision box size=0.11 0.12 0.049; visual box size=0.11 0.12 0.049
- link act1Seg5helper_shape: mass 0.0003 -> 0.0005949999999999999; geometry collision cylinder length=0.11 radius=0.06; visual cylinder length=0.11 radius=0.06
- link act1Seg6: mass 0.3 -> 0.595; geometry collision box size=0.11 0.12 0.049; visual box size=0.11 0.12 0.049
- link act1Seg6helper_shape: mass 0.0003 -> 0.0005949999999999999; geometry collision cylinder length=0.12 radius=0.055; visual cylinder length=0.12 radius=0.055
- link act1Seg7: mass 0.3 -> 0.595; geometry collision box size=0.11 0.12 0.049; visual box size=0.11 0.12 0.049
- link act1Seg7helper_shape: mass 0.0003 -> 0.0005949999999999999; geometry collision cylinder length=0.11 radius=0.06; visual cylinder length=0.11 radius=0.06
- link act1Seg8: mass 0.3 -> 0.595; geometry collision box size=0.11 0.12 0.049; visual box size=0.11 0.12 0.049
- link act1Seg8helper_shape: mass 0.0003 -> 0.0005949999999999999; geometry collision cylinder length=0.12 radius=0.055; visual cylinder length=0.12 radius=0.055
- link act1Seg9: mass 0.3 -> 0.595; geometry collision box size=0.11 0.12 0.049; visual box size=0.11 0.12 0.049
- link act1Seg9helper_shape: mass 0.0003 -> 0.0005949999999999999; geometry collision cylinder length=0.11 radius=0.06; visual cylinder length=0.11 radius=0.06
Joints:
- joint act0Seg0_to_act0Seg1_ax0: limit lower=-0.785398 upper=0.785398 effort=100 velocity=3 -> lower=0 upper=0 effort=100 velocity=3; origin xyz=0 0 0.0375 rpy=0 0 0 -> xyz=0 0 0.0245 rpy=0 0 0
- joint act0Seg0_to_act0Seg1_ax0helper_shape: origin xyz=0 0 0.0375 rpy=0 0 0 -> xyz=0 0 0.0245 rpy=0 0 0
- joint act0Seg10_to_act0Seg11_ax0: limit lower=-0.785398 upper=0.785398 effort=100 velocity=3 -> lower=0 upper=0 effort=100 velocity=3; origin xyz=0 0 0.075 rpy=0 0 0 -> xyz=0 0 0.049 rpy=0 0 0
- joint act0Seg10_to_act0Seg11_ax0helper_shape: origin xyz=0 0 0.075 rpy=0 0 0 -> xyz=0 0 0.049 rpy=0 0 0
- joint act0Seg11_to_act0Seg12_ax1: origin xyz=0 0 0.075 rpy=0 0 0 -> xyz=0 0 0.049 rpy=0 0 0
- joint act0Seg11_to_act0Seg12_ax1helper_shape: origin xyz=0 0 0.075 rpy=0 0 0 -> xyz=0 0 0.049 rpy=0 0 0
- joint act0Seg12_to_act0Seg13_ax0: limit lower=-0.785398 upper=0.785398 effort=100 velocity=3 -> lower=0 upper=0 effort=100 velocity=3; origin xyz=0 0 0.075 rpy=0 0 0 -> xyz=0 0 0.049 rpy=0 0 0
- joint act0Seg12_to_act0Seg13_ax0helper_shape: origin xyz=0 0 0.075 rpy=0 0 0 -> xyz=0 0 0.049 rpy=0 0 0
- joint act0Seg13_to_act0Seg14_ax1: origin xyz=0 0 0.075 rpy=0 0 0 -> xyz=0 0 0.049 rpy=0 0 0
- joint act0Seg13_to_act0Seg14_ax1helper_shape: origin xyz=0 0 0.075 rpy=0 0 0 -> xyz=0 0 0.049 rpy=0 0 0
- joint act0Seg14_to_act0Seg15_ax0: limit lower=-0.785398 upper=0.785398 effort=100 velocity=3 -> lower=0 upper=0 effort=100 velocity=3; origin xyz=0 0 0.075 rpy=0 0 0 -> xyz=0 0 0.049 rpy=0 0 0
- joint act0Seg14_to_act0Seg15_ax0helper_shape: origin xyz=0 0 0.075 rpy=0 0 0 -> xyz=0 0 0.049 rpy=0 0 0
- joint act0Seg15_to_act0Seg16_ax1: origin xyz=0 0 0.075 rpy=0 0 0 -> xyz=0 0 0.049 rpy=0 0 0
- joint act0Seg15_to_act0Seg16_ax1helper_shape: origin xyz=0 0 0.075 rpy=0 0 0 -> xyz=0 0 0.049 rpy=0 0 0
- joint act0Seg16_to_act0Seg17_ax0: limit lower=-0.785398 upper=0.785398 effort=100 velocity=3 -> lower=0 upper=0 effort=100 velocity=3; origin xyz=0 0 0.075 rpy=0 0 0 -> xyz=0 0 0.049 rpy=0 0 0
- joint act0Seg16_to_act0Seg17_ax0helper_shape: origin xyz=0 0 0.075 rpy=0 0 0 -> xyz=0 0 0.049 rpy=0 0 0
- joint act0Seg17_to_act0Seg18_ax1: origin xyz=0 0 0.075 rpy=0 0 0 -> xyz=0 0 0.049 rpy=0 0 0
- joint act0Seg17_to_act0Seg18_ax1helper_shape: origin xyz=0 0 0.075 rpy=0 0 0 -> xyz=0 0 0.049 rpy=0 0 0
- joint act0Seg18_to_act0Seg19_ax0: limit lower=-0.785398 upper=0.785398 effort=100 velocity=3 -> lower=0 upper=0 effort=100 velocity=3; origin xyz=0 0 0.075 rpy=0 0 0 -> xyz=0 0 0.049 rpy=0 0 0
- joint act0Seg18_to_act0Seg19_ax0helper_shape: origin xyz=0 0 0.075 rpy=0 0 0 -> xyz=0 0 0.049 rpy=0 0 0
- joint act0Seg19_to_act0Seg20_ax1: origin xyz=0 0 0.075 rpy=0 0 0 -> xyz=0 0 0.049 rpy=0 0 0
- joint act0Seg19_to_act0Seg20_ax1helper_shape: origin xyz=0 0 0.075 rpy=0 0 0 -> xyz=0 0 0.049 rpy=0 0 0
- joint act0Seg1_to_act0Seg2_ax1: origin xyz=0 0 0.075 rpy=0 0 0 -> xyz=0 0 0.049 rpy=0 0 0
- joint act0Seg1_to_act0Seg2_ax1helper_shape: origin xyz=0 0 0.075 rpy=0 0 0 -> xyz=0 0 0.049 rpy=0 0 0
- joint act0Seg20_to_act1Seg0_ax1: origin xyz=0 0 0.0375 rpy=0 0 0 -> xyz=0 0 0.0245 rpy=0 0 0
- joint act0Seg2_to_act0Seg3_ax0: limit lower=-0.785398 upper=0.785398 effort=100 velocity=3 -> lower=0 upper=0 effort=100 velocity=3; origin xyz=0 0 0.075 rpy=0 0 0 -> xyz=0 0 0.049 rpy=0 0 0
- joint act0Seg2_to_act0Seg3_ax0helper_shape: origin xyz=0 0 0.075 rpy=0 0 0 -> xyz=0 0 0.049 rpy=0 0 0
- joint act0Seg3_to_act0Seg4_ax1: origin xyz=0 0 0.075 rpy=0 0 0 -> xyz=0 0 0.049 rpy=0 0 0
- joint act0Seg3_to_act0Seg4_ax1helper_shape: origin xyz=0 0 0.075 rpy=0 0 0 -> xyz=0 0 0.049 rpy=0 0 0
- joint act0Seg4_to_act0Seg5_ax0: limit lower=-0.785398 upper=0.785398 effort=100 velocity=3 -> lower=0 upper=0 effort=100 velocity=3; origin xyz=0 0 0.075 rpy=0 0 0 -> xyz=0 0 0.049 rpy=0 0 0
- joint act0Seg4_to_act0Seg5_ax0helper_shape: origin xyz=0 0 0.075 rpy=0 0 0 -> xyz=0 0 0.049 rpy=0 0 0
- joint act0Seg5_to_act0Seg6_ax1: origin xyz=0 0 0.075 rpy=0 0 0 -> xyz=0 0 0.049 rpy=0 0 0
- joint act0Seg5_to_act0Seg6_ax1helper_shape: origin xyz=0 0 0.075 rpy=0 0 0 -> xyz=0 0 0.049 rpy=0 0 0
- joint act0Seg6_to_act0Seg7_ax0: limit lower=-0.785398 upper=0.785398 effort=100 velocity=3 -> lower=0 upper=0 effort=100 velocity=3; origin xyz=0 0 0.075 rpy=0 0 0 -> xyz=0 0 0.049 rpy=0 0 0
- joint act0Seg6_to_act0Seg7_ax0helper_shape: origin xyz=0 0 0.075 rpy=0 0 0 -> xyz=0 0 0.049 rpy=0 0 0
- joint act0Seg7_to_act0Seg8_ax1: origin xyz=0 0 0.075 rpy=0 0 0 -> xyz=0 0 0.049 rpy=0 0 0
- joint act0Seg7_to_act0Seg8_ax1helper_shape: origin xyz=0 0 0.075 rpy=0 0 0 -> xyz=0 0 0.049 rpy=0 0 0
- joint act0Seg8_to_act0Seg9_ax0: limit lower=-0.785398 upper=0.785398 effort=100 velocity=3 -> lower=0 upper=0 effort=100 velocity=3; origin xyz=0 0 0.075 rpy=0 0 0 -> xyz=0 0 0.049 rpy=0 0 0
- joint act0Seg8_to_act0Seg9_ax0helper_shape: origin xyz=0 0 0.075 rpy=0 0 0 -> xyz=0 0 0.049 rpy=0 0 0
- joint act0Seg9_to_act0Seg10_ax1: origin xyz=0 0 0.075 rpy=0 0 0 -> xyz=0 0 0.049 rpy=0 0 0
- joint act0Seg9_to_act0Seg10_ax1helper_shape: origin xyz=0 0 0.075 rpy=0 0 0 -> xyz=0 0 0.049 rpy=0 0 0
- joint act1Seg0_to_act1Seg1_ax0: limit lower=-0.785398 upper=0.785398 effort=100 velocity=3 -> lower=0 upper=0 effort=100 velocity=3; origin xyz=0 0 0.0375 rpy=0 0 0 -> xyz=0 0 0.0245 rpy=0 0 0
- joint act1Seg0_to_act1Seg1_ax0helper_shape: origin xyz=0 0 0.0375 rpy=0 0 0 -> xyz=0 0 0.0245 rpy=0 0 0
- joint act1Seg10_to_act1Seg11_ax0: limit lower=-0.785398 upper=0.785398 effort=100 velocity=3 -> lower=0 upper=0 effort=100 velocity=3; origin xyz=0 0 0.075 rpy=0 0 0 -> xyz=0 0 0.049 rpy=0 0 0
- joint act1Seg10_to_act1Seg11_ax0helper_shape: origin xyz=0 0 0.075 rpy=0 0 0 -> xyz=0 0 0.049 rpy=0 0 0
- joint act1Seg11_to_act1Seg12_ax1: origin xyz=0 0 0.075 rpy=0 0 0 -> xyz=0 0 0.049 rpy=0 0 0
- joint act1Seg11_to_act1Seg12_ax1helper_shape: origin xyz=0 0 0.075 rpy=0 0 0 -> xyz=0 0 0.049 rpy=0 0 0
- joint act1Seg12_to_act1Seg13_ax0: limit lower=-0.785398 upper=0.785398 effort=100 velocity=3 -> lower=0 upper=0 effort=100 velocity=3; origin xyz=0 0 0.075 rpy=0 0 0 -> xyz=0 0 0.049 rpy=0 0 0
- joint act1Seg12_to_act1Seg13_ax0helper_shape: origin xyz=0 0 0.075 rpy=0 0 0 -> xyz=0 0 0.049 rpy=0 0 0
- joint act1Seg13_to_act1Seg14_ax1: origin xyz=0 0 0.075 rpy=0 0 0 -> xyz=0 0 0.049 rpy=0 0 0
- joint act1Seg13_to_act1Seg14_ax1helper_shape: origin xyz=0 0 0.075 rpy=0 0 0 -> xyz=0 0 0.049 rpy=0 0 0
- joint act1Seg14_to_act1Seg15_ax0: limit lower=-0.785398 upper=0.785398 effort=100 velocity=3 -> lower=0 upper=0 effort=100 velocity=3; origin xyz=0 0 0.075 rpy=0 0 0 -> xyz=0 0 0.049 rpy=0 0 0
- joint act1Seg14_to_act1Seg15_ax0helper_shape: origin xyz=0 0 0.075 rpy=0 0 0 -> xyz=0 0 0.049 rpy=0 0 0
- joint act1Seg15_to_act1Seg16_ax1: origin xyz=0 0 0.075 rpy=0 0 0 -> xyz=0 0 0.049 rpy=0 0 0
- joint act1Seg15_to_act1Seg16_ax1helper_shape: origin xyz=0 0 0.075 rpy=0 0 0 -> xyz=0 0 0.049 rpy=0 0 0
- joint act1Seg16_to_act1Seg17_ax0: limit lower=-0.785398 upper=0.785398 effort=100 velocity=3 -> lower=0 upper=0 effort=100 velocity=3; origin xyz=0 0 0.075 rpy=0 0 0 -> xyz=0 0 0.049 rpy=0 0 0
- joint act1Seg16_to_act1Seg17_ax0helper_shape: origin xyz=0 0 0.075 rpy=0 0 0 -> xyz=0 0 0.049 rpy=0 0 0
- joint act1Seg17_to_act1Seg18_ax1: origin xyz=0 0 0.075 rpy=0 0 0 -> xyz=0 0 0.049 rpy=0 0 0
- joint act1Seg17_to_act1Seg18_ax1helper_shape: origin xyz=0 0 0.075 rpy=0 0 0 -> xyz=0 0 0.049 rpy=0 0 0
- joint act1Seg18_to_act1Seg19_ax0: limit lower=-0.785398 upper=0.785398 effort=100 velocity=3 -> lower=0 upper=0 effort=100 velocity=3; origin xyz=0 0 0.075 rpy=0 0 0 -> xyz=0 0 0.049 rpy=0 0 0
- joint act1Seg18_to_act1Seg19_ax0helper_shape: origin xyz=0 0 0.075 rpy=0 0 0 -> xyz=0 0 0.049 rpy=0 0 0
- joint act1Seg19_to_act1Seg20_ax1: origin xyz=0 0 0.075 rpy=0 0 0 -> xyz=0 0 0.049 rpy=0 0 0
- joint act1Seg19_to_act1Seg20_ax1helper_shape: origin xyz=0 0 0.075 rpy=0 0 0 -> xyz=0 0 0.049 rpy=0 0 0
- joint act1Seg1_to_act1Seg2_ax1: origin xyz=0 0 0.075 rpy=0 0 0 -> xyz=0 0 0.049 rpy=0 0 0
- joint act1Seg1_to_act1Seg2_ax1helper_shape: origin xyz=0 0 0.075 rpy=0 0 0 -> xyz=0 0 0.049 rpy=0 0 0
- joint act1Seg2_to_act1Seg3_ax0: limit lower=-0.785398 upper=0.785398 effort=100 velocity=3 -> lower=0 upper=0 effort=100 velocity=3; origin xyz=0 0 0.075 rpy=0 0 0 -> xyz=0 0 0.049 rpy=0 0 0
- joint act1Seg2_to_act1Seg3_ax0helper_shape: origin xyz=0 0 0.075 rpy=0 0 0 -> xyz=0 0 0.049 rpy=0 0 0
- joint act1Seg3_to_act1Seg4_ax1: origin xyz=0 0 0.075 rpy=0 0 0 -> xyz=0 0 0.049 rpy=0 0 0
- joint act1Seg3_to_act1Seg4_ax1helper_shape: origin xyz=0 0 0.075 rpy=0 0 0 -> xyz=0 0 0.049 rpy=0 0 0
- joint act1Seg4_to_act1Seg5_ax0: limit lower=-0.785398 upper=0.785398 effort=100 velocity=3 -> lower=0 upper=0 effort=100 velocity=3; origin xyz=0 0 0.075 rpy=0 0 0 -> xyz=0 0 0.049 rpy=0 0 0
- joint act1Seg4_to_act1Seg5_ax0helper_shape: origin xyz=0 0 0.075 rpy=0 0 0 -> xyz=0 0 0.049 rpy=0 0 0
- joint act1Seg5_to_act1Seg6_ax1: origin xyz=0 0 0.075 rpy=0 0 0 -> xyz=0 0 0.049 rpy=0 0 0
- joint act1Seg5_to_act1Seg6_ax1helper_shape: origin xyz=0 0 0.075 rpy=0 0 0 -> xyz=0 0 0.049 rpy=0 0 0
- joint act1Seg6_to_act1Seg7_ax0: limit lower=-0.785398 upper=0.785398 effort=100 velocity=3 -> lower=0 upper=0 effort=100 velocity=3; origin xyz=0 0 0.075 rpy=0 0 0 -> xyz=0 0 0.049 rpy=0 0 0
- joint act1Seg6_to_act1Seg7_ax0helper_shape: origin xyz=0 0 0.075 rpy=0 0 0 -> xyz=0 0 0.049 rpy=0 0 0
- joint act1Seg7_to_act1Seg8_ax1: origin xyz=0 0 0.075 rpy=0 0 0 -> xyz=0 0 0.049 rpy=0 0 0
- joint act1Seg7_to_act1Seg8_ax1helper_shape: origin xyz=0 0 0.075 rpy=0 0 0 -> xyz=0 0 0.049 rpy=0 0 0
- joint act1Seg8_to_act1Seg9_ax0: limit lower=-0.785398 upper=0.785398 effort=100 velocity=3 -> lower=0 upper=0 effort=100 velocity=3; origin xyz=0 0 0.075 rpy=0 0 0 -> xyz=0 0 0.049 rpy=0 0 0
- joint act1Seg8_to_act1Seg9_ax0helper_shape: origin xyz=0 0 0.075 rpy=0 0 0 -> xyz=0 0 0.049 rpy=0 0 0
- joint act1Seg9_to_act1Seg10_ax1: origin xyz=0 0 0.075 rpy=0 0 0 -> xyz=0 0 0.049 rpy=0 0 0
- joint act1Seg9_to_act1Seg10_ax1helper_shape: origin xyz=0 0 0.075 rpy=0 0 0 -> xyz=0 0 0.049 rpy=0 0 0
